File: hardware/Kicad/proyecto.papu/proyecto.papu.kicad_sch (KiCad schematic)
At the start: 19 parts, among them J1 Conn_01x04, J2 Conn_01x03, J3 Screw_Terminal_01x02, J4 Screw_Terminal_01x02, J5 Screw_Terminal_01x02, SW1 SW_Nidec_CAS-120A1, SW2 SW_MEC_5E, U1 DRV8833_MODULE, U2 L7805

Commit message: se termino pcb
Connections:
- net +12V: now also U1.4 (VCC)
- net 12v: no longer names the net of J5.1 (Pin_1), SW1.2 (B)
- net 12v: no longer U1.4 (VCC)
- net 3v renamed +3.3V
- no-connect marks 0 -> 3
Other:
- note added: "+12V"
